File: fancyfins/led_grouped.kicad_sch (KiCad schematic)
At the start: 5 parts, among them U8 L78L05_SOT89

Commit message: fixed led symbol
Connections:
- net DO: now also D15.1 (DO); no longer D15.4 (DO)
- net GND: now also D15.2 (VSS); no longer D15.1 (VSS)
- net at D5.1 (DO): now also D15.4 (DIN); no longer D15.2 (DIN)
