File: fancyfins/frodo_fancyfins.kicad_pcb (KiCad board)
At the start: 2 copper layers, 140 x 115 mm, 102 parts, among them J3 TC2050, U1 AZ1117-5.0, U10 L78L05_SOT89, U11 W25Q128JVP, U12 L78L05_SOT89, U13 L78L05_SOT89, U14 L78L05_SOT89, U15 L78L05_SOT89, U16 L78L05_SOT89, U2 AZ1117-3.3, U3 STM32F103RCTx, U4 MCP2562-E-SN, U5 TPD4E1U06, U6 L78L05_SOT89, U7 L78L05_SOT89, U8 L78L05_SOT89, U9 L78L05_SOT89, Y1 8MHz 12pF

Commit message: finished routing for fin board
Parts:
- removed the C16 at (184.7, 99.7)
- removed the C17 at (187.1, 100.5)
- removed the C8 at (196.2, 111.7)
- removed the R7 at (188.1, 118.3)
- removed the U5 at (197.7, 113.0)
- added C10: 22u, Capacitor_SMD:C_0805_2012Metric_Pad1.18x1.45mm_HandSolder, F.Cu at (178.2, 81.6)
- added C12: 100n, Capacitor_SMD:C_0402_1005Metric, F.Cu at (199.2, 90.3)
- added C2: 100n, Capacitor_SMD:C_0402_1005Metric, F.Cu at (208.2, 66.3)
- added C20: 1u, Capacitor_SMD:C_0402_1005Metric, F.Cu at (182.4, 96.8)
- added C21: 1u, Capacitor_SMD:C_0402_1005Metric, F.Cu at (183.2, 100.0)
- added C7: 100n, Capacitor_SMD:C_0402_1005Metric, F.Cu at (197.6, 83.2)
- added C9: 10u, Capacitor_SMD:C_0603_1608Metric_Pad1.08x0.95mm_HandSolder, F.Cu at (178.1, 88.5)
- added JP1: SolderJumper_3_Open, Jumper:SolderJumper-3_P1.3mm_Open_RoundedPad1.0x1.5mm, B.Cu at (209.8, 74.5)
- added R10: 22, Resistor_SMD:R_0402_1005Metric, F.Cu at (199.3, 87.6)
- added R11: 22, Resistor_SMD:R_0402_1005Metric, F.Cu at (199.3, 88.7)
- added R5: 4k7, Resistor_SMD:R_0603_1608Metric, F.Cu at (191.4, 79.1)
- added U3: TXB0102DCU, Package_SO:VSSOP-8_2.3x2mm_P0.5mm, F.Cu at (196.8, 80.4)
- added U4: AZ1117-3.3, Package_TO_SOT_SMD:SOT-223-3_TabPin2, F.Cu at (173.6, 84.5)
- added U7: TPD4E1U06, Package_TO_SOT_SMD:SOT-563, F.Cu at (201.2, 90.5)
- C1: value 100n -> 330n; footprint Capacitor_SMD:C_0402_1005Metric_Pad0.74x0.62mm_HandSolder -> Capacitor_SMD:C_0402_1005Metric
- C19: renamed from C15; footprint Capacitor_SMD:C_0402_1005Metric_Pad0.74x0.62mm_HandSolder -> Capacitor_SMD:C_0402_1005Metric
- C3: value 22u -> 100n; footprint Capacitor_SMD:C_0805_2012Metric_Pad1.18x1.45mm_HandSolder -> Capacitor_SMD:C_0402_1005Metric_Pad0.74x0.62mm_HandSolder
- C5: value 10u -> 22u; footprint Capacitor_SMD:C_0603_1608Metric_Pad1.08x0.95mm_HandSolder -> Capacitor_SMD:C_0805_2012Metric_Pad1.18x1.45mm_HandSolder
- C6: value 22u -> 100n; footprint Capacitor_SMD:C_0805_2012Metric_Pad1.18x1.45mm_HandSolder -> Capacitor_SMD:C_0402_1005Metric
- D1: value SS34 -> SK34
- R1: value 10k -> 680; footprint Resistor_SMD:R_0402_1005Metric -> Resistor_SMD:R_0603_1608Metric_Pad0.98x0.95mm_HandSolder
- R3: value 680 -> 10k; footprint Resistor_SMD:R_0603_1608Metric_Pad0.98x0.95mm_HandSolder -> Resistor_SMD:R_0402_1005Metric
- R4: value 10k -> 4k7; footprint Resistor_SMD:R_0402_1005Metric -> Resistor_SMD:R_0603_1608Metric
- TP1, TP2, TP3, TP4: moved to B.Cu
- U1: value AZ1117-5.0 -> 78L05S; footprint Package_TO_SOT_SMD:SOT-223-3_TabPin2 -> Package_TO_SOT_SMD:SOT-23
- U2: value AZ1117-3.3 -> AZ1117CH-3.3TRG1
- moved U1 99.0 mm to (208.3, 68.5)
- moved R1 90.7 mm to (123.2, 92.8), turned to -90 degrees
- moved R3 77.3 mm to (195.6, 83.2), turned to 180 degrees
- moved R13 73.9 mm to (178.8, 105.4), turned to 90 degrees
- moved R12 72.2 mm to (178.8, 107.4), turned to 90 degrees
- moved C3 62.5 mm to (180.2, 98.5), turned to 180 degrees
- moved U2 59.2 mm to (116.5, 91.3), turned to 90 degrees
- moved C1 52.0 mm to (207.9, 70.8), turned to 180 degrees
- moved C5 51.2 mm to (121.1, 89.3), turned to -90 degrees
- moved R2 32.8 mm to (188.2, 87.0), turned to -90 degrees
- moved J3 28.9 mm to (207.6, 90.5), turned to 180 degrees
- moved R8 27.5 mm to (199.2, 91.8), turned to 0 degrees
- moved R9 18.6 mm to (180.4, 100.0), turned to -90 degrees
- moved C6 16.3 mm to (196.8, 77.3), turned to 180 degrees
- moved C4 12.1 mm to (118.0, 96.5), turned to 180 degrees
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- renumbered C7 to C11, C9 to C13, C10 to C14, C11 to C15, C12 to C16, C13 to C17, C14 to C18, C18 to C22, C19 to C23, C20 to C24, C21 to C25, C23 to C26, C24 to C27, C25 to C28, C26 to C29, C27 to C30, C22 to C31, C28 to C32, C29 to C33, C30 to C34, C31 to C35, C32 to C36, C33 to C37, C34 to C38, C35 to C39, C2 to C4, C36 to C40, C37 to C41, C38 to C42, C39 to C43, C40 to C44, C4 to C8, R10 to R12, R11 to R13, R12 to R14, R5 to R6, R6 to R7, U8 to U10, U9 to U11, U10 to U12, U11 to U13, U12 to U14, U13 to U15, U14 to U16, U15 to U17, U16 to U18, U3 to U5, U4 to U6, U6 to U8, U7 to U9
Connections:
- C1 pad 1: NRST -> GND
- C1 pad 2: GND -> v_main
- C3 pad 1: +5V -> NRST
- C6 pad 1: +3.3V -> GND
- C6 pad 2: GND -> +3.3V
- J1 pad 4: CAN_L_OUT -> CAN_L_IN
- J1 pad 8: CAN_H_OUT -> CAN_H_IN
- J2 pad 1: P_SDA -> Net-(J2-Pin_1)
- J2 pad 2: P_SCL -> Net-(J2-Pin_2)
- J2 pad 4: P_A_Out -> unconnected-(J2-Pin_4-Pad4)
- J2 pad 8: +3.3V -> Net-(J2-Pin_8)
- J3 pad 1: NRST -> Net-(J3-Pin_1)
- J3 pad 10: +5V -> unconnected-(J3-Pin_10-Pad10)
- J3 pad 6: Net-(J3-Pin_6) -> /J1-SWCLK
- J3 pad 9: +5V -> unconnected-(J3-Pin_9-Pad9)
- R1 pad 1: +3.3V -> Net-(D2-K)
- R1 pad 2: P_SCL -> GND
- R2 pad 1: +3.3V -> GND
- R2 pad 2: P_SDA -> BOOT0
- R3 pad 1: Net-(D2-K) -> Net-(U3-OE)
- R4 pad 1: GND -> +3.3V
- R4 pad 2: BOOT0 -> P_SCL
- R8 pad 1: SWO -> SWDIO
- R8 pad 2: /J1-SWO -> /J1-SWDIO
- R9 pad 1: Net-(J3-Pin_6) -> NRST
- R9 pad 2: SWCLK -> Net-(J3-Pin_1)
- U1 pad 1: GND -> Net-(J2-Pin_8)
- U1 pad 2: +5V -> v_main
- U1 pad 3: v_main -> GND
- U2 pad 2: +3.3V -> +5V
- U2 pad 3: +5V -> v_main
- U5 pad 29: P_SCL -> unconnected-(U5-PB10-Pad29)
- U5 pad 30: P_SDA -> unconnected-(U5-PB11-Pad30)
- U5 pad 44: unconnected-(U3-PA11-Pad44) -> CAN_RX
- U5 pad 45: unconnected-(U3-PA12-Pad45) -> CAN_TX
- U5 pad 58: unconnected-(U3-PB6-Pad58) -> P_SCL
- U5 pad 59: unconnected-(U3-PB7-Pad59) -> P_SDA
- U5 pad 61: CAN_RX -> unconnected-(U5-PB8-Pad61)
- U5 pad 62: CAN_TX -> unconnected-(U5-PB9-Pad62)
Routing:
- net v_main: track 4.56 -> 143.4 mm
- net VDsense: track 98.1 -> 17.8 mm, vias 4 -> 2
- net GND: track 80.1 -> 143.8 mm, vias 148 -> 381
- net Net-(J3-Pin_1): track 0.00 -> 62.2 mm, vias 0 -> 2
- net +5V: track 142.2 -> 82.7 mm
- net SWCLK: track 63.1 -> 5.23 mm, vias 4 -> 0
- net +3.3V: track 262.8 -> 209.2 mm, vias 4 -> 5
- net P_A_Out: track 52.7 -> 0.00 mm
- net VD: track 305.1 -> 256.5 mm
- net SWDIO: track 47.8 -> 2.54 mm, vias 2 -> 0
- net P_SDA: track 57.2 -> 15.3 mm
- net SWO: track 47.8 -> 6.09 mm, vias 4 -> 0
- net P_SCL: track 55.8 -> 14.5 mm
- net Net-(J2-Pin_1): track 0.00 -> 41.0 mm
- net Net-(J2-Pin_2): track 0.00 -> 36.8 mm
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- added copper zone on F.Cu, net +3.3V
- added copper zone on F.Cu, net +5V
Other:
- outline, holes or cut-outs redrawn
- board text added: "RAPID Fin Board v2"

Commit message: some changes according to manu, added connector board
Parts:
- added G***: LOGO, hephaistos:rapid_logo, F.Cu at (216.2, 145.0)
- D4: value D_Schottky -> SK34; footprint Diode_SMD:D_SOD-123F -> Diode_SMD:D_SMA
- F1: value 1A -> 3A
- FB1: footprint Inductor_SMD:L_0603_1608Metric_Pad1.05x0.95mm_HandSolder -> Inductor_SMD:L_0402_1005Metric
- moved R7 10.0 mm to (107.0, 87.9)
- moved C11 9.75 mm to (108.4, 84.7)
- moved C4 9.75 mm to (127.8, 96.5)
- moved C5 9.75 mm to (130.8, 89.3)
- moved C8 9.75 mm to (116.0, 88.0)
- moved D1 9.75 mm to (111.8, 93.1)
- moved D2 9.75 mm to (132.9, 89.3)
- moved U2 9.75 mm to (126.2, 91.3)
- moved U6 9.75 mm to (111.8, 88.0)
- moved R1 9.75 mm to (132.9, 92.8)
- moved D4 5.41 mm to (111.8, 96.8)
- moved C43 4.90 mm to (217.5, 135.4)
- moved C44 4.90 mm to (219.4, 135.4)
- moved U18 4.90 mm to (218.4, 132.0)
- moved C22 4.50 mm to (217.8, 43.0)
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Connections:
- J2 pad 3: GND -> unconnected-(J2-Pin_3-Pad3)
- J2 pad 5: unconnected-(J2-Pin_5-Pad5) -> GND
Routing:
- net VD: track 256.5 -> 243.2 mm
- net +5V: track 82.7 -> 72.8 mm
- net v_main: track 143.4 -> 133.7 mm
- net Net-(D1-A): track 19.1 -> 28.8 mm
- net CAN_TX: track 114.0 -> 104.4 mm
- net CAN_L_IN: track 18.5 -> 28.0 mm
- net CAN_H_IN: track 17.9 -> 27.4 mm
- net CAN_RX: track 117.1 -> 107.6 mm
- net +3.3V: track 209.2 -> 199.8 mm
- net Net-(D4-A): track 1.81 -> 6.68 mm
- net Net-(D23-VDD): track 13.7 -> 17.3 mm
- net Net-(D5-VDD): track 14.1 -> 16.9 mm
- net VDsense: track 17.8 -> 16.3 mm
- net charging_voltage: track 20.6 -> 19.4 mm
- net GND: track 143.8 -> 144.8 mm, vias 381 -> 366
Other:
- outline, holes or cut-outs redrawn
- board text added: "JLCJLCJLCJLC"
