File: fin_flex_cable/fin_flex_cable.kicad_sch (KiCad schematic)
At the start: 4 parts, among them J5 Conn_02x04_Top_Bottom, J6 Conn_02x04_Top_Bottom, J7 Conn_02x04_Top_Bottom

Commit message: finished layout, added a bunch of footprints, fixed outer form
Parts:
- J5, J6, J7: footprint (none) -> fancyfins:009159008801906
Changed lines of the file:
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@@
 			)
 		)
-		(property "Footprint" ""
+		(property "Footprint" "fancyfins:009159008801906"
 			(at 121.92 59.69 0)
 			(effects
@@
 			)
 		)
-		(property "Footprint" ""
+		(property "Footprint" "fancyfins:009159008801906"
 			(at 45.72 59.69 0)
 			(effects
@@
 			)
 		)
-		(property "Footprint" ""
+		(property "Footprint" "fancyfins:009159008801906"
 			(at 83.82 59.69 0)
 			(effects

Commit message: finished routing for fin board
Connections:
- net v_charge: no longer J5.6 (Pin_6), J6.6 (Pin_6), J7.6 (Pin_6), J8.6 (Pin_6)
- new net v_main: J5.6 (Pin_6), J6.6 (Pin_6), J7.6 (Pin_6), J8.6 (Pin_6)
Changed lines of the file:
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@@
-		(color 0 0 0 0)
-	)
-	(junction
-		(at 91.44 52.07)
-		(diameter 0)
 		(color 0 0 0 0)
 	)
@@
 	(wire
 		(pts
-			(xy 91.44 52.07) (xy 91.44 57.15)
-		)
-		(stroke
-			(width 0)
-			(type default)
-		)
-	)
-	(wire
-		(pts
 			(xy 53.34 59.69) (xy 57.15 59.69)
 		)
@@
 	(wire
 		(pts
-			(xy 91.44 52.07) (xy 93.98 52.07)
+			(xy 57.15 52.07) (xy 93.98 52.07)
 		)
 		(stroke
@@
 	(wire
 		(pts
-			(xy 91.44 49.53) (xy 91.44 52.07)
+			(xy 91.44 49.53) (xy 91.44 57.15)
 		)
 		(stroke
@@
 		)
 	)
-	(wire
-		(pts
-			(xy 57.15 52.07) (xy 91.44 52.07)
-		)
-		(stroke
-			(width 0)
-			(type default)
-		)
-	)
