File: sensor_pcb/sensor_pcb.kicad_sch (KiCad schematic)
At the start: 2 parts, among them IC1 WSEN-PDUS_2513130810402, J7 Conn_02x04_Top_Bottom

Commit message: some changes according to manu, added connector board
Connections:
- net at J7.3 (Pin_3): no longer IC1.3
- net at J7.4 (Pin_4): no longer IC1.4
- net at J7.5 (Pin_5): now also IC1.3
- net at J7.6 (Pin_6): now also IC1.4
Changed lines of the file:
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@@
 	(paper "A4")
 	(no_connect
+		(at 87.63 64.77)
+	)
+	(no_connect
 		(at 101.6 43.18)
 	)
 	(no_connect
-		(at 100.33 62.23)
+		(at 87.63 67.31)
 	)
 	(no_connect
@@
 		(at 100.33 64.77)
 	)
-	(no_connect
-		(at 100.33 59.69)
-	)
-	(wire
-		(pts
-			(xy 101.6 48.26) (xy 105.41 48.26)
+	(wire
+		(pts
+			(xy 101.6 48.26) (xy 106.68 48.26)
+		)
+		(stroke
+			(width 0)
+			(type default)
+		)
+	)
+	(wire
+		(pts
+			(xy 85.09 48.26) (xy 85.09 52.07)
 		)
 		(stroke
@@
 	(wire
 		(pts
-			(xy 85.09 48.26) (xy 85.09 67.31)
+			(xy 101.6 54.61) (xy 101.6 59.69)
+		)
+		(stroke
+			(width 0)
+			(type default)
+		)
+	)
+	(wire
+		(pts
+			(xy 82.55 45.72) (xy 82.55 54.61)
 		)
 		(stroke
@@
 	(wire
 		(pts
-			(xy 87.63 64.77) (xy 82.55 64.77)
-		)
-		(stroke
-			(width 0)
-			(type default)
-		)
-	)
-	(wire
-		(pts
 			(xy 77.47 59.69) (xy 87.63 59.69)
 		)
@@
 	(wire
 		(pts
-			(xy 85.09 67.31) (xy 87.63 67.31)
-		)
-		(stroke
-			(width 0)
-			(type default)
-		)
-	)
-	(wire
-		(pts
 			(xy 80.01 43.18) (xy 80.01 62.23)
 		)
@@
 	(wire
 		(pts
-			(xy 100.33 67.31) (xy 105.41 67.31)
+			(xy 100.33 67.31) (xy 106.68 67.31)
 		)
 		(stroke
@@
 	(wire
 		(pts
-			(xy 105.41 48.26) (xy 105.41 67.31)
-		)
-		(stroke
-			(width 0)
-			(type default)
-		)
-	)
-	(wire
-		(pts
-			(xy 82.55 64.77) (xy 82.55 45.72)
+			(xy 104.14 62.23) (xy 100.33 62.23)
+		)
+		(stroke
+			(width 0)
+			(type default)
+		)
+	)
+	(wire
+		(pts
+			(xy 104.14 52.07) (xy 104.14 62.23)
+		)
+		(stroke
+			(width 0)
+			(type default)
+		)
+	)
+	(wire
+		(pts
+			(xy 106.68 48.26) (xy 106.68 67.31)
+		)
+		(stroke
+			(width 0)
+			(type default)
+		)
+	)
+	(wire
+		(pts
+			(xy 85.09 52.07) (xy 104.14 52.07)
+		)
+		(stroke
+			(width 0)
+			(type default)
+		)
+	)
+	(wire
+		(pts
+			(xy 82.55 54.61) (xy 101.6 54.61)
+		)
+		(stroke
+			(width 0)
+			(type default)
+		)
+	)
+	(wire
+		(pts
+			(xy 100.33 59.69) (xy 101.6 59.69)
 		)
 		(stroke
@@
 			)
 		)
-		(property "Datasheet" "chrome-extension://efaidnbmnnnibpcajpcglclefindmkaj/https://www.we-online.com/components/products/datasheet/2513130810301.pdf"
+		(property "Datasheet" "https://www.we-online.com/components/products/datasheet/2513130810301.pdf"
 			(at 93.98 45.72 0)
 			(effects
